File: fixed_mcu/led.kicad_sch (KiCad schematic)
At the start: 20 parts

Commit message: Implemented board layout
Parts:
- renumbered D22 to L1, D31 to L10, D32 to L11, D33 to L12, D34 to L13, D35 to L14, D36 to L15, D37 to L16, D38 to L17, D39 to L18, D40 to L19, D23 to L2, D41 to L20, D24 to L3, D25 to L4, D26 to L5, D27 to L6, D28 to L7, D29 to L8, D30 to L9
