File: fixed_mcu/switches.kicad_sch (KiCad schematic)
At the start: 40 parts, among them SW10 CherryMX, SW11 CherryMX, SW12 CherryMX, SW13 CherryMX, SW14 CherryMX, SW15 CherryMX, SW16 CherryMX, SW17 CherryMX, SW18 CherryMX, SW19 CherryMX, SW2 CherryMX, SW20 CherryMX, SW21 CherryMX, SW3 CherryMX, SW4 CherryMX, SW5 CherryMX, SW6 CherryMX, SW7 CherryMX, SW8 CherryMX, SW9 CherryMX

Commit message: Implemented board layout
Parts:
- D10, D11, D12, D13, D14, D15, D16, D17, D18, D19, D2, D20, D21, D3, D4, D5, D6, D7, D8, D9: footprint (none) -> Diode_SMD:D_0805_2012Metric_Pad1.15x1.40mm_HandSolder
- SW1: renamed from SW2; footprint (none) -> ScottoKeebs_Hotswap:Hotswap_MX_1.00u
- SW10: renamed from SW11; footprint (none) -> ScottoKeebs_Hotswap:Hotswap_MX_1.00u
- SW11: renamed from SW12; footprint (none) -> ScottoKeebs_Hotswap:Hotswap_MX_1.00u
- SW12: renamed from SW13; footprint (none) -> ScottoKeebs_Hotswap:Hotswap_MX_1.00u
- SW13: renamed from SW14; footprint (none) -> ScottoKeebs_Hotswap:Hotswap_MX_1.00u
- SW14: renamed from SW15; footprint (none) -> ScottoKeebs_Hotswap:Hotswap_MX_1.00u
- SW15: renamed from SW16; footprint (none) -> ScottoKeebs_Hotswap:Hotswap_MX_1.00u
- SW16: renamed from SW17; footprint (none) -> ScottoKeebs_Hotswap:Hotswap_MX_1.00u
- SW17: renamed from SW18; footprint (none) -> ScottoKeebs_Hotswap:Hotswap_MX_1.00u
- SW18: renamed from SW19; footprint (none) -> ScottoKeebs_Hotswap:Hotswap_MX_1.00u
- SW19: renamed from SW20; footprint (none) -> ScottoKeebs_Hotswap:Hotswap_MX_1.00u
- SW2: renamed from SW3; footprint (none) -> ScottoKeebs_Hotswap:Hotswap_MX_1.00u
- SW20: renamed from SW21; footprint (none) -> ScottoKeebs_Hotswap:Hotswap_MX_1.00u
- SW3: renamed from SW4; footprint (none) -> ScottoKeebs_Hotswap:Hotswap_MX_1.00u
- SW4: renamed from SW5; footprint (none) -> ScottoKeebs_Hotswap:Hotswap_MX_1.00u
- SW5: renamed from SW6; footprint (none) -> ScottoKeebs_Hotswap:Hotswap_MX_1.00u
- SW6: renamed from SW7; footprint (none) -> ScottoKeebs_Hotswap:Hotswap_MX_1.00u
- SW7: renamed from SW8; footprint (none) -> ScottoKeebs_Hotswap:Hotswap_MX_1.00u
- SW8: renamed from SW9; footprint (none) -> ScottoKeebs_Hotswap:Hotswap_MX_1.00u
- SW9: renamed from SW10; footprint (none) -> ScottoKeebs_Hotswap:Hotswap_MX_1.00u
